File: _autosave-pulp.kicad_pcb (KiCad board)
At the start: 2 copper layers, 40.8 x 81.5 mm, 42 parts, among them J1 Conn_Coaxial, J2 Conn_01x02_Pin, J3 Conn_01x02_Pin, J4 Conn_01x03_Pin, J5 Conn_01x03_Pin, J6 Conn_01x06_Pin, U1 HMC5883L, U2 RP2040, U3 MAX-M8Q, U4 AP7361C-33E, X2 ASE-12.0MHz

Commit message: finalized a lot of sub-modules
Parts:
- added C5: 4.7uF, Capacitor_SMD:C_0201_0603Metric, F.Cu at (63.4, 111.5)
- added C6: 1uF, Capacitor_SMD:C_0201_0603Metric, F.Cu at (58.1, 111.2)
- added C7: 4.7uF, Capacitor_SMD:C_0201_0603Metric, F.Cu at (63.5, 107.3)
- added J7: USB_C_Receptacle, Connector_USB:USB_C_Receptacle_CNCTech_C-ARA1-AK51X, F.Cu at (65.9, 116.8)
- moved U4 50.1 mm to (58.6, 105.3), turned to 90 degrees
- moved C16 20.4 mm to (71.7, 101.3)
- moved C20 20.4 mm to (71.7, 97.5)
- moved C21 20.4 mm to (71.7, 99.3)
- moved C22 20.4 mm to (71.7, 100.3)
- moved C24 20.4 mm to (71.7, 98.3)
- moved C25 20.4 mm to (71.7, 96.6)
- moved C26 20.4 mm to (71.7, 102.2)
- moved C27 20.4 mm to (71.7, 103.2)
- moved C28 20.4 mm to (71.7, 104.1)
- moved J4 13.9 mm to (84.9, 68.5)
- moved J5 13.9 mm to (84.9, 73.5)
- moved C19 4.31 mm to (72.0, 87.8)
- moved R18 3.11 mm to (70.0, 87.9)
- moved R17 2.23 mm to (67.5, 86.4)
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Routing:
- net +5V: track 0.00 -> 11.6 mm
- net /RP2040/1V1: track 8.53 -> 0.00 mm
- net Net-(U2-QSPI_SD1): track 3.11 -> 0.05 mm
- net +3V3: track 27.4 -> 24.4 mm, vias 2 -> 0
- net Net-(U2-QSPI_SD2): track 2.90 -> 0.00 mm
- net Net-(U2-QSPI_SD0): track 2.71 -> 0.00 mm
- net Net-(U2-QSPI_SCLK): track 2.53 -> 0.00 mm
- net Net-(U2-QSPI_SD3): track 2.34 -> 0.06 mm
- net /USB_D+: track 1.43 -> 0.00 mm
- net /USB_D-: track 1.38 -> 0.00 mm
