File: MAX_8C.kicad_sch (KiCad schematic)
At the start: 6 parts, among them J1 Conn_Coaxial, U3 MAX-M8Q

Commit message: finalized a lot of sub-modules
Parts:
- C3, C4: footprint (none) -> Capacitor_SMD:C_0201_0603Metric
- J1: footprint (none) -> Connector_Coaxial:SMA_Amphenol_901-143_Horizontal
- L1: footprint (none) -> Inductor_SMD:L_0201_0603Metric
- R3: footprint (none) -> Resistor_SMD:R_0201_0603Metric
Changed lines of the file:
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@@
       (effects (font (size 1.27 1.27)) (justify left))
     )
-    (property "Footprint" "" (at 96.2152 27.94 0)
+    (property "Footprint" "Capacitor_SMD:C_0201_0603Metric" (at 96.2152 27.94 0)
       (effects (font (size 1.27 1.27)) hide)
     )
@@
       (effects (font (size 1.27 1.27)) (justify left))
     )
-    (property "Footprint" "" (at 127 46.99 0)
+    (property "Footprint" "Inductor_SMD:L_0201_0603Metric" (at 127 46.99 0)
       (effects (font (size 1.27 1.27)) hide)
     )
@@
       (effects (font (size 1.27 1.27)) (justify left))
     )
-    (property "Footprint" "" (at 120.3452 40.64 0)
+    (property "Footprint" "Capacitor_SMD:C_0201_0603Metric" (at 120.3452 40.64 0)
       (effects (font (size 1.27 1.27)) hide)
     )
@@
       (effects (font (size 1.27 1.27)))
     )
-    (property "Footprint" "" (at 111.76 33.528 90)
+    (property "Footprint" "Resistor_SMD:R_0201_0603Metric" (at 111.76 33.528 90)
       (effects (font (size 1.27 1.27)) hide)
     )
@@
       (effects (font (size 1.27 1.27)) (justify left))
     )
-    (property "Footprint" "" (at 137.16 50.8 0)
+    (property "Footprint" "Connector_Coaxial:SMA_Amphenol_901-143_Horizontal" (at 137.16 50.8 0)
       (effects (font (size 1.27 1.27)) hide)
     )

Commit message: NO ERC ERRORS!!!!
Connections:
- net SCL: no longer names the net of U3.17 (SCL)
- net SDA: no longer names the net of U3.16 (SDA)
- no-connect marks 0 -> 7
Changed lines of the file:
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@@
   (junction (at 92.71 33.02) (diameter 0) (color 0 0 0 0)
   )
-  (wire (pts (xy 76.2 50.8) (xy 82.55 50.8))
+  (no_connect (at 76.2 50.8))
+  (no_connect (at 76.2 55.88))
+  (no_connect (at 116.84 58.42))
+  (no_connect (at 76.2 58.42))
+  (no_connect (at 76.2 48.26))
+  (no_connect (at 76.2 60.96))
+  (no_connect (at 116.84 45.72))
+  (wire (pts (xy 76.2 48.26) (xy 82.55 48.26))
     (stroke (width 0) (type default))
   )
@@
     (stroke (width 0) (type default))
   )
+  (wire (pts (xy 76.2 50.8) (xy 82.55 50.8))
+    (stroke (width 0) (type default))
+  )
   (wire (pts (xy 95.25 26.67) (xy 95.25 27.94))
     (stroke (width 0) (type default))
@@
     (stroke (width 0) (type default))
   )
-  (wire (pts (xy 92.71 20.32) (xy 95.25 20.32))
+  (wire (pts (xy 113.03 45.72) (xy 116.84 45.72))
     (stroke (width 0) (type default))
   )
-  (wire (pts (xy 76.2 48.26) (xy 82.55 48.26))
+  (wire (pts (xy 113.03 58.42) (xy 116.84 58.42))
+    (stroke (width 0) (type default))
+  )
+  (wire (pts (xy 92.71 20.32) (xy 95.25 20.32))
     (stroke (width 0) (type default))
   )
@@
     (stroke (width 0) (type default))
   )
+  (wire (pts (xy 76.2 55.88) (xy 82.55 55.88))
+    (stroke (width 0) (type default))
+  )
   (wire (pts (xy 115.57 31.75) (xy 119.38 31.75))
+    (stroke (width 0) (type default))
+  )
+  (wire (pts (xy 76.2 58.42) (xy 82.55 58.42))
+    (stroke (width 0) (type default))
+  )
+  (wire (pts (xy 76.2 60.96) (xy 82.55 60.96))
     (stroke (width 0) (type default))
   )
@@
     (effects (font (size 1.27 1.27)) (justify right))
   )
-  (hierarchical_label "SCL" (shape input) (at 76.2 50.8 180) (fields_autoplaced)
-    (effects (font (size 1.27 1.27)) (justify right))
-  )
-  (hierarchical_label "SDA" (shape input) (at 76.2 48.26 180) (fields_autoplaced)
-    (effects (font (size 1.27 1.27)) (justify right))
-  )

Commit message: finished pcb layout
Parts:
- J1: footprint Connector_Coaxial:SMA_Amphenol_901-143_Horizontal -> Connector_Coaxial:U.FL_Molex_MCRF_73412-0110_Vertical
