File: RP2040.kicad_sch (KiCad schematic)
At the start: 25 parts, among them U1 RP2040, X1 ASE-12.0MHz

Commit message: finalized a lot of sub-modules
Connections:
- net LED_R (GPIO_15): now reaches U1.18 (GPIO15)
- net LED_G (GPIO_16): now reaches U1.27 (GPIO16)
- net LED_B (GPIO_17): now reaches U1.28 (GPIO17)
- net SWCLK: no longer names the net of U1.24 (SWCLK)
- net SWD: no longer names the net of U1.25 (SWD)
- no-connect marks 1 -> 3
Changed lines of the file:
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@@
   (junction (at 151.13 21.59) (diameter 0) (color 0 0 0 0)
   )
+  (no_connect (at 85.09 110.49))
   (no_connect (at 87.63 97.79))
+  (no_connect (at 85.09 107.95))
   (wire (pts (xy 130.81 21.59) (xy 135.89 21.59))
     (stroke (width 0) (type default))
@@
     (stroke (width 0) (type default))
   )
+  (wire (pts (xy 143.51 80.01) (xy 173.99 80.01))
+    (stroke (width 0) (type default))
+  )
   (wire (pts (xy 52.07 41.91) (xy 92.71 41.91))
     (stroke (width 0) (type default))
@@
     (stroke (width 0) (type default))
   )
+  (wire (pts (xy 85.09 110.49) (xy 92.71 110.49))
+    (stroke (width 0) (type default))
+  )
   (wire (pts (xy 127 34.29) (xy 128.27 34.29))
     (stroke (width 0) (type default))
@@
     (stroke (width 0) (type default))
   )
+  (wire (pts (xy 85.09 107.95) (xy 92.71 107.95))
+    (stroke (width 0) (type default))
+  )
   (wire (pts (xy 140.97 21.59) (xy 146.05 21.59))
     (stroke (width 0) (type default))
@@
     (stroke (width 0) (type default))
   )
+  (wire (pts (xy 143.51 85.09) (xy 173.99 85.09))
+    (stroke (width 0) (type default))
+  )
   (wire (pts (xy 111.76 25.4) (xy 111.76 34.29))
     (stroke (width 0) (type default))
@@
   )
   (wire (pts (xy 113.03 34.29) (xy 115.57 34.29))
+    (stroke (width 0) (type default))
+  )
+  (wire (pts (xy 143.51 82.55) (xy 173.99 82.55))
     (stroke (width 0) (type default))
   )
@@
     (effects (font (size 1.27 1.27)) (justify left))
   )
+  (hierarchical_label "LED_B (GPIO_17)" (shape output) (at 173.99 85.09 0) (fields_autoplaced)
+    (effects (font (size 1.27 1.27)) (justify left))
+  )
   (hierarchical_label "QSPI_SS" (shape input) (at 74.93 59.69 180) (fields_autoplaced)
     (effects (font (size 1.27 1.27)) (justify right))
@@
     (effects (font (size 1.27 1.27)) (justify right))
   )
-  (hierarchical_label "SWCLK" (shape input) (at 92.71 107.95 180) (fields_autoplaced)
-    (effects (font (size 1.27 1.27)) (justify right))
-  )
   (hierarchical_label "I2C 0 SCL" (shape bidirectional) (at 173.99 97.79 0) (fields_autoplaced)
     (effects (font (size 1.27 1.27)) (justify left))
   )
+  (hierarchical_label "LED_G (GPIO_16)" (shape output) (at 173.99 82.55 0) (fields_autoplaced)
+    (effects (font (size 1.27 1.27)) (justify left))
+  )
   (hierarchical_label "GPIO 3" (shape bidirectional) (at 173.99 49.53 0) (fields_autoplaced)
     (effects (font (size 1.27 1.27)) (justify left))
@@
     (effects (font (size 1.27 1.27)) (justify right))
   )
+  (hierarchical_label "LED_R (GPIO_15)" (shape output) (at 173.99 80.01 0) (fields_autoplaced)
+    (effects (font (size 1.27 1.27)) (justify left))
+  )
   (hierarchical_label "QSPI_0" (shape bidirectional) (at 71.12 64.77 180) (fields_autoplaced)
     (effects (font (size 1.27 1.27)) (justify right))
   )
-  (hierarchical_label "SWD" (shape bidirectional) (at 92.71 110.49 180) (fields_autoplaced)
-    (effects (font (size 1.27 1.27)) (justify right))
-  )

Commit message: NO ERC ERRORS!!!!
Connections:
- no-connect marks 3 -> 16
Changed lines of the file:
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@@
   )
   (no_connect (at 85.09 110.49))
+  (no_connect (at 153.67 102.87))
   (no_connect (at 87.63 97.79))
+  (no_connect (at 153.67 118.11))
+  (no_connect (at 153.67 69.85))
   (no_connect (at 85.09 107.95))
+  (no_connect (at 153.67 113.03))
+  (no_connect (at 153.67 62.23))
+  (no_connect (at 153.67 105.41))
+  (no_connect (at 153.67 110.49))
+  (no_connect (at 153.67 100.33))
+  (no_connect (at 153.67 67.31))
+  (no_connect (at 153.67 74.93))
+  (no_connect (at 153.67 64.77))
+  (no_connect (at 153.67 92.71))
+  (no_connect (at 153.67 115.57))
   (wire (pts (xy 130.81 21.59) (xy 135.89 21.59))
     (stroke (width 0) (type default))
@@
     (stroke (width 0) (type default))
   )
+  (wire (pts (xy 143.51 64.77) (xy 153.67 64.77))
+    (stroke (width 0) (type default))
+  )
   (wire (pts (xy 34.29 31.75) (xy 36.83 31.75))
     (stroke (width 0) (type default))
@@
     (stroke (width 0) (type default))
   )
+  (wire (pts (xy 143.51 113.03) (xy 153.67 113.03))
+    (stroke (width 0) (type default))
+  )
   (wire (pts (xy 135.89 29.21) (xy 140.97 29.21))
     (stroke (width 0) (type default))
@@
     (stroke (width 0) (type default))
   )
+  (wire (pts (xy 143.51 105.41) (xy 153.67 105.41))
+    (stroke (width 0) (type default))
+  )
+  (wire (pts (xy 143.51 74.93) (xy 153.67 74.93))
+    (stroke (width 0) (type default))
+  )
   (wire (pts (xy 143.51 77.47) (xy 173.99 77.47))
     (stroke (width 0) (type default))
@@
     (stroke (width 0) (type default))
   )
+  (wire (pts (xy 143.51 110.49) (xy 153.67 110.49))
+    (stroke (width 0) (type default))
+  )
   (wire (pts (xy 135.89 21.59) (xy 140.97 21.59))
     (stroke (width 0) (type default))
@@
     (stroke (width 0) (type default))
   )
+  (wire (pts (xy 143.51 69.85) (xy 153.67 69.85))
+    (stroke (width 0) (type default))
+  )
+  (wire (pts (xy 143.51 118.11) (xy 153.67 118.11))
+    (stroke (width 0) (type default))
+  )
+  (wire (pts (xy 143.51 62.23) (xy 153.67 62.23))
+    (stroke (width 0) (type default))
+  )
   (wire (pts (xy 127 16.51) (xy 127 21.59))
     (stroke (width 0) (type default))
@@
     (stroke (width 0) (type default))
   )
+  (wire (pts (xy 143.51 115.57) (xy 153.67 115.57))
+    (stroke (width 0) (type default))
+  )
   (wire (pts (xy 34.29 73.66) (xy 34.29 80.01))
     (stroke (width 0) (type default))
@@
     (stroke (width 0) (type default))
   )
+  (wire (pts (xy 143.51 102.87) (xy 153.67 102.87))
+    (stroke (width 0) (type default))
+  )
+  (wire (pts (xy 143.51 100.33) (xy 153.67 100.33))
+    (stroke (width 0) (type default))
+  )
+  (wire (pts (xy 143.51 67.31) (xy 153.67 67.31))
+    (stroke (width 0) (type default))
+  )
   (wire (pts (xy 146.05 29.21) (xy 151.13 29.21))
     (stroke (width 0) (type default))
@@
     (stroke (width 0) (type default))
   )
+  (wire (pts (xy 143.51 92.71) (xy 153.67 92.71))
+    (stroke (width 0) (type default))
+  )

Commit message: finished pcb layout
Parts:
- renumbered C13 to C15, C14 to C16, C12 to C17, C11 to C18, C10 to C19, C1 to C20, C2 to C21, C3 to C22, C4 to C23, C5 to C24, C6 to C25, C7 to C26, C8 to C27, C9 to C28, R2 to R10, R1 to R11, R9 to R12, R8 to R13, R7 to R14, R6 to R15, R5 to R16, R3 to R17, R4 to R18, U1 to U2, X1 to X2
Connections:
- net USB_D+: now also R17.1; no longer R18.1, R18.2, U2.46 (USB_DM)
- net USB_D-: now also R18.2; no longer R17.1, R17.2, U2.47 (USB_DP)
- new net: R17.2, U2.47 (USB_DP)
- new net: R18.1, U2.46 (USB_DM)
