File: qmc5883L.kicad_sch (KiCad schematic)
At the start: 5 parts, among them U1 HMC5883L

Commit message: NO ERC ERRORS!!!!
Connections:
- no-connect marks 0 -> 8
Changed lines of the file:
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@@
   (junction (at 74.93 26.67) (diameter 0) (color 0 0 0 0)
   )
+  (no_connect (at 71.12 54.61))
+  (no_connect (at 29.21 44.45))
+  (no_connect (at 71.12 57.15))
+  (no_connect (at 29.21 41.91))
+  (no_connect (at 71.12 62.23))
+  (no_connect (at 29.21 39.37))
+  (no_connect (at 29.21 46.99))
+  (no_connect (at 29.21 36.83))
   (wire (pts (xy 64.77 39.37) (xy 74.93 39.37))
     (stroke (width 0) (type default))
@@
     (stroke (width 0) (type default))
   )
+  (wire (pts (xy 39.37 39.37) (xy 29.21 39.37))
+    (stroke (width 0) (type default))
+  )
   (wire (pts (xy 26.67 59.69) (xy 39.37 59.69))
     (stroke (width 0) (type default))
   )
+  (wire (pts (xy 39.37 44.45) (xy 29.21 44.45))
+    (stroke (width 0) (type default))
+  )
   (wire (pts (xy 64.77 41.91) (xy 74.93 41.91))
+    (stroke (width 0) (type default))
+  )
+  (wire (pts (xy 64.77 54.61) (xy 71.12 54.61))
     (stroke (width 0) (type default))
   )
@@
   )
   (wire (pts (xy 87.63 49.53) (xy 85.09 49.53))
+    (stroke (width 0) (type default))
+  )
+  (wire (pts (xy 64.77 62.23) (xy 71.12 62.23))
+    (stroke (width 0) (type default))
+  )
+  (wire (pts (xy 64.77 57.15) (xy 71.12 57.15))
     (stroke (width 0) (type default))
   )
@@
     (stroke (width 0) (type default))
   )
+  (wire (pts (xy 39.37 41.91) (xy 29.21 41.91))
+    (stroke (width 0) (type default))
+  )
   (wire (pts (xy 26.67 52.07) (xy 26.67 57.15))
     (stroke (width 0) (type default))
@@
     (stroke (width 0) (type default))
   )
+  (wire (pts (xy 39.37 46.99) (xy 29.21 46.99))
+    (stroke (width 0) (type default))
+  )
   (wire (pts (xy 64.77 49.53) (xy 68.58 49.53))
     (stroke (width 0) (type default))
@@
     (stroke (width 0) (type default))
   )
+  (wire (pts (xy 39.37 36.83) (xy 29.21 36.83))
+    (stroke (width 0) (type default))
+  )
